File: Hardware/Qwiic Distance Sensor - VL53L1X.brd (EAGLE design)
At the start: 25.4 x 25.4 mm, 45 parts, among them J2 SMD, J3 PTH, J4 SMD, U2 VL53L1XSMD

Commit message: Moving examples for lib. Adding I2C capture logs.
Parts:
- U2: value VL53L1XSMD -> VL53L1X
Changed lines of the file:
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@@
 <element name="U$1" library="SparkX" package="SPARKX-MEDIUM" value="SPARKX-LOGO4" x="12.7" y="23.495"/>
 <element name="J5" library="SparkFun-Connectors" package="1X01_NO_SILK" value="" x="16.51" y="1.27"/>
-<element name="U2" library="VL53L1X" package="VL53L1X" value="VL53L1XSMD" x="12.7" y="12.7"/>
+<element name="U2" library="VL53L1X" package="VL53L1X" value="VL53L1X" x="12.7" y="12.7"/>
 <element name="R1" library="SparkFun-Resistors" package="0603" value="10k" x="7.62" y="12.7" rot="R90">
 <attribute name="PROD_ID" value="RES-00824" x="7.62" y="12.7" size="1.778" layer="27" font="vector" ratio="15" rot="R90" display="off"/>
