File: Hardware/Qwiic Distance Sensor - VL53L1X.sch (EAGLE design)
At the start: 26 parts, among them J2 SMD, J3 PTH, J4 SMD, U2 VL53L1XSMD

Commit message: Moving examples for lib. Adding I2C capture logs.
Parts:
- U2: value VL53L1XSMD -> VL53L1X
Changed lines of the file:
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@@
 <part name="U$1" library="SparkX" deviceset="SPARKX-LOGO" device="4"/>
 <part name="J5" library="SparkFun-Connectors" deviceset="CONN_01" device="PTH_NO_SILK_YES_STOP"/>
-<part name="U2" library="VL53L1X" deviceset="VL53L1X" device="SMD"/>
+<part name="U2" library="VL53L1X" deviceset="VL53L1X" device="SMD" value="VL53L1X"/>
 <part name="R1" library="SparkFun-Resistors" deviceset="10KOHM" device="-0603-1/10W-1%" value="10k"/>
 <part name="R2" library="SparkFun-Resistors" deviceset="10KOHM" device="-0603-1/10W-1%" value="10k"/>
